File: kicad/mrb-fcs/mrb-fcs.kicad_sch (KiCad schematic)
At the start: 43 parts, among them J1 Phoenix Contact 1988804, J2 USB Mini B Jack, Q1 BSS138K, SW1 FSM4JSMATR, U1 AP63203WU, U2 ESP32-C6-WROOM-1, U3 TLC59284, U4 TLC59284

Commit message: Update schematic, complete PCB
Parts:
- added C10: 22uF, Capacitor_SMD:C_0805_2012Metric, symbol Device:C
- added C9: 0.1uF, Capacitor_SMD:C_0805_2012Metric, symbol Device:C
- added D9: YELLOW, LED_SMD:LED_0805_2012Metric, symbol Device:LED
- added R11: 1k, Resistor_SMD:R_0805_2012Metric, symbol Device:R_US
Connections:
- net +3.3V: now also C10.1, C9.1
- net BLINK_COLON: now also U2.16 (GPIO18); no longer U2.17 (GPIO19)
- net GND: now also C10.2, C9.2, D9.1 (K)
- net DISP1_1_F: now reaches DISP1.18 (DIG1_F)
- net DISP1_1_F: now also U4.20 (OUT15); no longer U3.10 (OUT5)
- net DISP1_1_G: now reaches DISP1.17 (DIG1_G)
- net DISP1_1_G: now also U4.19 (OUT14); no longer U3.11 (OUT6)
- net DISP1_1_DP: now reaches DISP1.4 (DIG1_DP)
- net DISP1_1_DP: now also U3.8 (OUT3); no longer U3.12 (OUT7)
- net DISP1_2_A: now reaches DISP1.11 (DIG2_A)
- net DISP1_2_A: now also U4.15 (OUT10); no longer U3.13 (OUT8)
- net DISP1_2_B: now reaches DISP1.10 (DIG2_B)
- net DISP1_2_B: now also U4.14 (OUT9); no longer U3.14 (OUT9)
- net DISP1_2_C: now reaches DISP1.8 (DIG2_C)
- net DISP1_2_C: now also U3.12 (OUT7); no longer U3.15 (OUT10)
- net DISP1_2_D: now reaches DISP1.6 (DIG2_D)
- net DISP1_2_D: now also U3.10 (OUT5); no longer U3.16 (OUT11)
- net DISP1_2_E: now reaches DISP1.5 (DIG2_E)
- net DISP1_2_E: now also U3.9 (OUT4); no longer U3.17 (OUT12)
- net DISP1_2_F: now reaches DISP1.12 (DIG2_F)
- net DISP1_2_F: now also U4.16 (OUT11); no longer U3.18 (OUT13)
- net DISP1_2_G: now reaches DISP1.7 (DIG2_G)
- net DISP1_2_G: now also U3.11 (OUT6); no longer U3.19 (OUT14)
- net BLANK: now reaches U2.18 (GPIO20)
- net BLANK: now also U3.21 (BLANK), U4.21 (BLANK); no longer U3.2 (SIN)
- net DISP1_2_DP: now reaches DISP1.9 (DIG2_DP)
- net DISP1_2_DP: now also U3.13 (OUT8); no longer U3.20 (OUT15)
- net LATCH: now reaches U3.4 (LAT), U4.4 (LAT)
- net LATCH: now also U2.19 (GPIO21); no longer U2.20 (GPIO22)
- net DISP1_1_A: now reaches DISP1.16 (DIG1_A)
- net DISP1_1_A: now also U4.18 (OUT13); no longer U3.5 (OUT0)
- net DISP1_1_B: now reaches DISP1.15 (DIG1_B)
- net DISP1_1_B: now also U4.17 (OUT12); no longer U3.6 (OUT1)
- net DISP1_1_C: now reaches DISP1.3 (DIG1_C), U3.7 (OUT2)
- net DISP1_1_D: now reaches DISP1.2 (DIG1_D)
- net DISP1_1_D: now also U3.6 (OUT1); no longer U3.8 (OUT3)
- net DISP1_1_E: now reaches DISP1.1 (DIG1_E)
- net DISP1_1_E: now also U3.5 (OUT0); no longer U3.9 (OUT4)
- net DISP2_1_A: now reaches U4.9 (OUT4)
- net DISP2_1_A: now also DISP2.16 (DIG1_A); no longer DISP2.1 (DIG1_E)
- net DISP2_2_B: now reaches DISP2.10 (DIG2_B)
- net DISP2_2_B: now also U4.5 (OUT0); no longer U4.14 (OUT9)
- net DISP2_1_D: now reaches U4.13 (OUT8)
- net DISP2_1_D: now also DISP2.2 (DIG1_D); no longer DISP2.11 (DIG2_A)
- net DISP2_2_F: now reaches DISP2.12 (DIG2_F)
- net DISP2_2_F: now also U4.7 (OUT2); no longer U4.18 (OUT13)
- net DISP2_1_B: now reaches DISP2.15 (DIG1_B)
- net DISP2_1_B: now also U4.8 (OUT3); no longer U4.6 (OUT1)
- net DISP2_1_F: now reaches U4.11 (OUT6)
- net DISP2_1_F: now also DISP2.18 (DIG1_F); no longer DISP2.17 (DIG1_G)
- net DISP2_1_G: now reaches U4.10 (OUT5)
- net DISP2_1_G: now also DISP2.17 (DIG1_G); no longer DISP2.18 (DIG1_F)
- net DISP2_1_C: now reaches DISP2.3 (DIG1_C)
- net DISP2_1_C: now also U3.14 (OUT9); no longer U4.7 (OUT2)
- net DISP2_1_DP: now reaches DISP2.4 (DIG1_DP)
- net DISP2_1_DP: now also U3.15 (OUT10); no longer U4.12 (OUT7)
- net DISP2_2_E: now reaches DISP2.5 (DIG2_E)
- net DISP2_2_E: now also U3.16 (OUT11); no longer U4.17 (OUT12)
- net DISP2_2_D: now reaches DISP2.6 (DIG2_D)
- net DISP2_2_D: now also U3.17 (OUT12); no longer U4.16 (OUT11)
- net DISP2_2_G: now reaches DISP2.7 (DIG2_G)
- net DISP2_2_G: now also U3.18 (OUT13); no longer U4.19 (OUT14)
- net DISP2_2_C: now reaches DISP2.8 (DIG2_C)
- net DISP2_2_C: now also U3.19 (OUT14); no longer U4.15 (OUT10)
- net DISP2_2_DP: now reaches DISP2.9 (DIG2_DP)
- net DISP2_2_DP: now also U3.20 (OUT15); no longer U4.20 (OUT15)
- net at U2.12 (GPIO11): now also R11.2
- new net: D9.2 (A), R11.1
- new net DISP2_1_E: DISP2.1 (DIG1_E), U4.12 (OUT7)
- new net DISP2_2_A: DISP2.11 (DIG2_A), U4.6 (OUT1)
- new net SCLK: U2.20 (GPIO22), U3.3 (SCLK), U4.3 (SCLK)
- new net SDO: U2.21 (GPIO23), U3.2 (SIN)
Other:
- moved on the sheet: C7, C8, DISP1, DISP2, R10, R7, R8, R9, U3, U4
